File: Diseño-PCB/Sistema Riego Inteligente/Sistema Riego Inteligente.kicad_sch (KiCad schematic)
At the start: 5 parts, among them U1 DEVKIT_V1_ESP32-WROOM-32, U2 DHT11

Commit message: Actualizo esquemático
Parts:
- added D1: 1N4007, Diode_THT:D_DO-41_SOD81_P10.16mm_Horizontal, symbol Diode:1N4007
- added J1: electroválvula, Connector_Phoenix_MC:PhoenixContact_MC_1,5_2-GF-3.5_1x02_P3.50mm_Horizontal_ThreadedFlange, symbol Connector_Generic:Conn_01x02
- renumbered K1 to U3
Connections:
- net GND: now also U3.5 (COM)
- net at U3.6 (NO): now also D1.1 (K), J1.2 (Pin_2)
- net S renamed RELE_CTRL
- new net +12V: D1.2 (A), J1.1 (Pin_1)
Other:
- moved on the sheet: DS1, R1, U2

Commit message: Completo ruteo y diseño de PCB
Parts:
- J1: footprint Connector_Phoenix_MC:PhoenixContact_MC_1,5_2-GF-3.5_1x02_P3.50mm_Horizontal_ThreadedFlange -> Connector_Phoenix_GMSTB:PhoenixContact_GMSTBA_2,5_2-G_1x02_P7.50mm_Horizontal
Other:
- moved on the sheet: D1, DS1, J1, R1, U1, U2, U3
